Commit message: feat: add robot mesh files

File: src/asr_sdm_universe/robot/asr_sdm_description/urdf/Robot.urdf (robot description, URDF)
Before this commit: robot Robot, 4 links, 3 joints
Links:
- added link l_cycloid_outter_motor_opposite_side003; visual mesh filename=package://asr_sdm_description/meshes/asr_sdm_v1_cycloid_out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
- added link l_cycloid_outter_motor_side003; visual mesh filename=package://asr_sdm_description/meshes/asr_sdm_v1_cycloid_out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
- added link l_screw_rotor_right001; visual mesh filename=package://asr_sdm_description/meshes/asr_sdm_v1_screw_rotor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
Joints:
- added joint l_cycloid_outter_motor_opposite_side001__to__l_cycloid_outter_motor_opposite_side003: type fixed, parent l_cycloid_outter_motor_opposite_side001, child l_cycloid_outter_motor_opposite_side003, origin xyz=0.0 0.0 0.0 rpy=0 0 0
- added joint l_cycloid_outter_motor_opposite_side003__to__l_cycloid_outter_motor_side003: type fixed, parent l_cycloid_outter_motor_opposite_side003, child l_cycloid_outter_motor_side003, origin xyz=0.0 0.0 0.0 rpy=0 0 0
- added joint l_cycloid_outter_motor_opposite_side003__to__l_screw_rotor_right001: type continuous, parent l_cycloid_outter_motor_opposite_side003, child l_screw_rotor_right001, origin xyz=0.0 0.0 0.0 rpy=0 0 0, axis 1 0 0
