Commit message: feat:add asr_sdm kinematic rviz simulation

File: src/asr_sdm_universe/robot/asr_sdm/urdf/asr_sdm.urdf.xacro (robot description, xacro)
@@ -6,4 +6,14 @@
   <xacro:property name="CONNECT_XYZ" value="-0.046790 -0.000087 -0.018248"/>
   <xacro:property name="CONNECT_RPY" value="1.5707963267948966 0 -1.5707963267948966"/>
+  <!-- ================= 最小运动学/刚体动力学参数 ================= -->
+  <!-- XM430-W350：初始仿真限制。机械角限位取较保守的 ±1 rad。 -->
+  <xacro:property name="SERVO_LOWER" value="-1.0"/>
+  <xacro:property name="SERVO_UPPER" value="1.0"/>
+  <xacro:property name="SERVO_EFFORT" value="4.0"/>
+  <xacro:property name="SERVO_VELOCITY" value="4.82"/>
+  <!-- 螺旋转子：缺少实际电机型号时采用的初始仿真值。 -->
+  <!-- 20.943951 rad/s = 200 rpm；0.10 N·m 仅为保守仿真上限。 -->
+  <xacro:property name="ROTOR_EFFORT" value="0.10"/>
+  <xacro:property name="ROTOR_VELOCITY" value="20.9439510239"/>
   <!-- ================= 单个节段 ================= -->
   <!-- 每节均包含主体和两个螺旋转子；末节不包含 A/Cross/B 关节单元。 -->
@@ -54,4 +64,5 @@
             <origin rpy="0 0 0" xyz="0.0 0.0 0.01275" />
             <axis xyz="0 0 1" />
+            <limit effort="${ROTOR_EFFORT}" velocity="${ROTOR_VELOCITY}" />
           </joint>
         <joint name="joint_screwdrive_segment_0__screw_rotor_right_0__${idx}" type="continuous">
@@ -60,13 +71,83 @@
             <origin rpy="0 0 0" xyz="0.0 0.0 0.0825" />
             <axis xyz="0 0 1" />
+            <limit effort="${ROTOR_EFFORT}" velocity="${ROTOR_VELOCITY}" />
+            <!-- 右转子位置、速度和加速度均与左转子反向。 -->
+            <mimic joint="joint_screwdrive_segment_0__screw_rotor_left_0__${idx}"
+                   multiplier="-1.0" offset="0.0" />
           </joint>
     <!-- A / Cross / B 关节单元，末节跳过。 -->
     <xacro:if value="${idx + 1 &lt; int(N)}">
             <link name="joint_unit_a_${idx}">
-                <visual><origin rpy="0 0 0" xyz="0 0 0" /><geometry><mesh filename="package://asr_sdm/meshes/joint_unit_a.stl" /></geometry><material name="mat_joint_unit_a_${idx}"><color rgba="0.678431 0.709804 0.741176 1" /></material></visual></link>
+              <!-- XM430-W350 与输出/从动侧安装附件的等效质量属性。 -->
+              <!-- 质量取 0.105 kg；惯量由 82 g STL 均匀分布结果按质量线性缩放。 -->
+              <inertial>
+                <mass value="0.105" />
+                <origin rpy="0 0 0" xyz="-0.000354695736 -0.0000183839643 0.0219250269" />
+                <inertia
+                  ixx="3.69265338786e-05"
+                  ixy="-2.40610257648e-08"
+                  ixz="2.33629298824e-07"
+                  iyy="4.06736219268e-05"
+                  iyz="-2.83212124166e-08"
+                  izz="2.47155849478e-05" />
+              </inertial>
+              <visual>
+                <origin rpy="0 0 0" xyz="0 0 0" />
+                <geometry>
+                  <mesh filename="package://asr_sdm/meshes/joint_unit_a.stl" />
+                </geometry>
+                <material name="mat_joint_unit_a_${idx}">
+                  <color rgba="0.678431 0.709804 0.741176 1" />
+                </material>
+              </visual>
+            </link>
             <link name="joint_unit_cross_${idx}">
-                <visual><origin rpy="0 0 0" xyz="0 0 0" /><geometry><mesh filename="package://asr_sdm/meshes/joint_unit_cross.stl" /></geometry><material name="mat_joint_unit_cross_${idx}"><color rgba="0.678431 0.709804 0.741176 1" /></material></visual></link>
+              <!-- 两个 FR12-H101K 正交连接及紧固件的等效质量属性。 -->
+              <!-- 质量取 0.020 kg；质心和惯量由组合 STL 的均匀质量分布计算。 -->
+              <inertial>
+                <mass value="0.020" />
+                <origin rpy="0 0 0" xyz="0.000313986224 -0.018982444334 0.019003452419" />
+                <inertia
+                  ixx="3.85136165390e-06"
+                  ixy="-2.56677722305e-08"
+                  ixz="7.13023772897e-13"
+                  iyy="5.90814768259e-06"
+                  iyz="-3.88597622857e-13"
+                  izz="3.85104301667e-06" />
+              </inertial>
+              <visual>
+                <origin rpy="0 0 0" xyz="0 0 0" />
+                <geometry>
+                  <mesh filename="package://asr_sdm/meshes/joint_unit_cross.stl" />
+                </geometry>
+                <material name="mat_joint_unit_cross_${idx}">
+                  <color rgba="0.678431 0.709804 0.741176 1" />
+                </material>
+              </visual>
+            </link>
             <link name="joint_unit_b_${idx}">
-                <visual><origin rpy="0 0 0" xyz="0 0 0" /><geometry><mesh filename="package://asr_sdm/meshes/joint_unit_b.stl" /></geometry><material name="mat_joint_unit_b_${idx}"><color rgba="0.678431 0.709804 0.741176 1" /></material></visual></link>
+              <!-- XM430-W350 与输出/从动侧安装附件的等效质量属性。 -->
+              <!-- 质量取 0.105 kg；惯量由 82 g STL 均匀分布结果按质量线性缩放。 -->
+              <inertial>
+                <mass value="0.105" />
+                <origin rpy="0 0 0" xyz="-0.0169779299 0.000139808905 -0.0186162548" />
+                <inertia
+                  ixx="2.36615114444e-05"
+                  ixy="1.11368664330e-07"
+                  ixz="-5.46313091894e-07"
+                  iyy="3.97164045384e-05"
+                  iyz="8.17139817483e-10"
+                  izz="3.57206534120e-05" />
+              </inertial>
+              <visual>
+                <origin rpy="0 0 0" xyz="0 0 0" />
+                <geometry>
+                  <mesh filename="package://asr_sdm/meshes/joint_unit_b.stl" />
+                </geometry>
+                <material name="mat_joint_unit_b_${idx}">
+                  <color rgba="0.678431 0.709804 0.741176 1" />
+                </material>
+              </visual>
+            </link>
             <joint name="joint_screwdrive_segment_0__joint_unit_a__${idx}" type="fixed">
                 <parent link="screwdrive_segment_${idx}" />
@@ -79,5 +160,5 @@
                 <origin rpy="-1.5707963267948966 0 -1.5707963267948966" xyz="-0.0190035 -8.38634e-05 0.0392499" />
                 <axis xyz="0 0 1" />
-                <limit effort="0.0" lower="-1.5707963267948966" upper="1.5707963267948966" velocity="0.0" />
+                <limit effort="${SERVO_EFFORT}" lower="${SERVO_LOWER}" upper="${SERVO_UPPER}" velocity="${SERVO_VELOCITY}" />
               </joint>
             <joint name="joint_joint_unit_cross__joint_unit_b__${idx}" type="revolute">
@@ -86,5 +167,5 @@
                 <origin rpy="-1.5707963267948968 0 1.5707963267948966" xyz="-0.018332 -0.03796 0.018873" />
                 <axis xyz="0 0 1" />
-                <limit effort="0.0" lower="-1.5707963267948966" upper="1.5707963267948966" velocity="0.0" />
+                <limit effort="${SERVO_EFFORT}" lower="${SERVO_LOWER}" upper="${SERVO_UPPER}" velocity="${SERVO_VELOCITY}" />
               </joint>
     </xacro:if>
@@ -105,5 +186,4 @@
     </xacro:if>
   </xacro:macro>
-  <!-- 根 link 保持自由；显示启动文件使用 world 到根 link 的静态 TF 调整朝向。 -->
   <xacro:snake_chain/>
 </robot>

Commit message: amend_robot_forward

File: src/asr_sdm_universe/robot/asr_sdm/urdf/asr_sdm.urdf.xacro (robot description, xacro)
@@ -32,5 +32,12 @@
               <inertia ixx="0.0008368145831015" ixy="3.348578885e-07" ixz="1.3959146972e-06" iyy="0.0008365215316531" iyz="4.092756065e-07" izz="0.0001491920058212" />
             </inertial>
-          <visual><origin rpy="0 0 0" xyz="0 0 0" /><geometry><mesh filename="package://asr_sdm/meshes/screwdrive_segment_0.stl" /></geometry><material name="mat_screwdrive_segment_${idx}"><color rgba="0.678431 0.709804 0.741176 1" /></material></visual></link>
+          <visual>
+              <origin rpy="0 0 0" xyz="0 0 0.08725" />
+              <geometry>
+                <cylinder length="0.1855000000000001" radius="0.03" />
+              </geometry>
+              <material name="mat_screwdrive_segment_${idx}"><color rgba="0.678431 0.709804 0.741176 1" /></material>
+            </visual>
+        </link>
         <link name="screw_rotor_left_${idx}">
             <collision>
@@ -45,5 +52,12 @@
               <inertia ixx="1.94327521911e-05" ixy="8.165e-13" ixz="-2.5e-15" iyy="1.94376384386e-05" iyz="-1.817e-13" izz="3.56879993201e-05" />
             </inertial>
-          <visual><origin rpy="0 0 0" xyz="0 0 0" /><geometry><mesh filename="package://asr_sdm/meshes/screw_rotor_left_0.stl" /></geometry><material name="mat_screw_rotor_left_${idx}"><color rgba="0.678431 0.709804 0.741176 1" /></material></visual></link>
+            <visual>
+              <origin rpy="0 0 0" xyz="0 0 0" />
+              <geometry>
+                <cylinder length="0.0255" radius="0.047" />
+              </geometry>
+              <material name="mat_screw_rotor_left_${idx}"><color rgba="0.5 0.5 0.5 1" /></material>
+            </visual>
+        </link>
         <link name="screw_rotor_right_${idx}">
             <collision>
@@ -58,5 +72,12 @@
               <inertia ixx="1.94322695895e-05" ixy="8.147e-13" ixz="5.3e-15" iyy="1.94371557899e-05" iyz="1.806e-13" izz="3.5687294149e-05" />
             </inertial>
-          <visual><origin rpy="0 0 0" xyz="0 0 0" /><geometry><mesh filename="package://asr_sdm/meshes/screw_rotor_right_0.stl" /></geometry><material name="mat_screw_rotor_right_${idx}"><color rgba="0.678431 0.709804 0.741176 1" /></material></visual></link>
+            <visual>
+              <origin rpy="0 0 0" xyz="0 0 0" />
+              <geometry>
+                <cylinder length="0.0255" radius="0.047" />
+              </geometry>
+              <material name="mat_screw_rotor_right_${idx}"><color rgba="0.5 0.5 0.5 1" /></material>
+            </visual>
+        </link>
         <joint name="joint_screwdrive_segment_0__screw_rotor_left_0__${idx}" type="continuous">
             <parent link="screwdrive_segment_${idx}" />
@@ -79,6 +100,4 @@
     <xacro:if value="${idx + 1 &lt; int(N)}">
             <link name="joint_unit_a_${idx}">
-              <!-- XM430-W350 与输出/从动侧安装附件的等效质量属性。 -->
-              <!-- 质量取 0.105 kg；惯量由 82 g STL 均匀分布结果按质量线性缩放。 -->
               <inertial>
                 <mass value="0.105" />
@@ -95,5 +114,5 @@
                 <origin rpy="0 0 0" xyz="0 0 0" />
                 <geometry>
-                  <mesh filename="package://asr_sdm/meshes/joint_unit_a.stl" />
+                  <box size="0.04 0.04 0.04" />
                 </geometry>
                 <material name="mat_joint_unit_a_${idx}">
@@ -103,6 +122,4 @@
             </link>
             <link name="joint_unit_cross_${idx}">
-              <!-- 两个 FR12-H101K 正交连接及紧固件的等效质量属性。 -->
-              <!-- 质量取 0.020 kg；质心和惯量由组合 STL 的均匀质量分布计算。 -->
               <inertial>
                 <mass value="0.020" />
@@ -119,5 +136,5 @@
                 <origin rpy="0 0 0" xyz="0 0 0" />
                 <geometry>
-                  <mesh filename="package://asr_sdm/meshes/joint_unit_cross.stl" />
+                  <box size="0.04 0.04 0.04" />
                 </geometry>
                 <material name="mat_joint_unit_cross_${idx}">
@@ -127,6 +144,4 @@
             </link>
             <link name="joint_unit_b_${idx}">
-              <!-- XM430-W350 与输出/从动侧安装附件的等效质量属性。 -->
-              <!-- 质量取 0.105 kg；惯量由 82 g STL 均匀分布结果按质量线性缩放。 -->
               <inertial>
                 <mass value="0.105" />
@@ -143,5 +158,5 @@
                 <origin rpy="0 0 0" xyz="0 0 0" />
                 <geometry>
-                  <mesh filename="package://asr_sdm/meshes/joint_unit_b.stl" />
+                  <box size="0.04 0.04 0.04" />
                 </geometry>
                 <material name="mat_joint_unit_b_${idx}">

File: src/asr_sdm_universe/robot/asr_sdm/urdf/asr_sdm_sensors.urdf.xacro (robot description, xacro)
@@ -1,4 +1,14 @@
 <?xml version="1.0"?>
 <robot xmlns:xacro="http://www.ros.org/wiki/xacro" name="asr_sdm_sensors">
-  <!-- 传感器和 Gazebo 插件将在此扩展。 -->
+  <!-- ================= ROOT BASE FRAME ================= -->
+  <!-- 'base' is the VINS body frame (published by odom_visualization) and is the
+       URDF root. The RPY here MUST match the static TF published by
+       tf2_ros static_transform_publisher in asr_sdm_description.launch.py
+       (yaml.robot_model.yaw_rad / pitch_rad). Currently: yaw=π, pitch=-π/2. -->
+  <link name="base"/>
+  <joint name="joint_base_to_screwdrive_segment_0" type="fixed">
+    <parent link="base"/>
+    <child link="screwdrive_segment_0"/>
+    <origin rpy="0 0 0" xyz="0 0 0"/>
+  </joint>
 </robot>

Commit message: fix: align the tf coordinate frames

File: src/asr_sdm_universe/robot/asr_sdm/urdf/asr_sdm.urdf.xacro (robot description, xacro)
@@ -187,3 +187,20 @@
   </xacro:macro>
   <xacro:snake_chain/>
+  <!-- VINS / 里程计坐标系 base：相机光轴沿 +Z（与 camera_pose_visual 一致）。 -->
+  <!-- ROS 机器人坐标系 base_link：前进方向 +X、左侧 +Y、上方 +Z。 -->
+  <!-- rpy (0, -π/2, π) 把 base +Z 映到 base_link +X，从而对齐相机框与机器人。 -->
+  <link name="base"/>
+  <joint name="base_to_base_link" type="fixed">
+    <parent link="base"/>
+    <child link="base_link"/>
+    <origin rpy="0 -1.5707963267948966 3.141592653589793" xyz="0 0 0"/>
+  </joint>
+  <!-- CAD 沿节段 +Z 建模，头部朝向为 -Z。 -->
+  <!-- 绕 Y 转 -π/2，使头部朝向变为 base_link +X。 -->
+  <link name="base_link"/>
+  <joint name="base_link_to_screwdrive_segment_0" type="fixed">
+    <parent link="base_link"/>
+    <child link="screwdrive_segment_0"/>
+    <origin rpy="0 -1.5707963267948966 0" xyz="0 0 0"/>
+  </joint>
 </robot>

Commit message: fix: realign coordinate frames in planning simulator

File: src/asr_sdm_universe/robot/asr_sdm/urdf/asr_sdm.urdf.xacro (robot description, xacro)
@@ -187,12 +187,10 @@
   </xacro:macro>
   <xacro:snake_chain/>
-  <!-- VINS / 里程计坐标系 base：相机光轴沿 +Z（与 camera_pose_visual 一致）。 -->
-  <!-- ROS 机器人坐标系 base_link：前进方向 +X、左侧 +Y、上方 +Z。 -->
-  <!-- rpy (0, -π/2, π) 把 base +Z 映到 base_link +X，从而对齐相机框与机器人。 -->
+  <!-- base 与控制器 / 2D Pose Estimate 一致：+X 朝前、+Y 朝左、+Z 朝上。 -->
   <link name="base"/>
   <joint name="base_to_base_link" type="fixed">
     <parent link="base"/>
     <child link="base_link"/>
-    <origin rpy="0 -1.5707963267948966 3.141592653589793" xyz="0 0 0"/>
+    <origin rpy="0 0 0" xyz="0 0 0"/>
   </joint>
   <!-- CAD 沿节段 +Z 建模，头部朝向为 -Z。 -->

Commit message: feat: refactor control para

File: src/asr_sdm_universe/robot/asr_sdm/urdf/asr_sdm.urdf.xacro (robot description, xacro)
@@ -72,7 +72,4 @@
             <axis xyz="0 0 1" />
             <limit effort="${ROTOR_EFFORT}" velocity="${ROTOR_VELOCITY}" />
-            <!-- 右转子位置、速度和加速度均与左转子反向。 -->
-            <mimic joint="joint_screwdrive_segment_0__screw_rotor_left_0__${idx}"
-                   multiplier="-1.0" offset="0.0" />
           </joint>
     <!-- A / Cross / B 关节单元，末节跳过。 -->
